File: Amplifier PCB.kicad_pcb (KiCad board)
At the start: 4 copper layers, 23 x 43 mm, 20 parts, among them J1 sma, J2 sma, J3 Screw_Terminal_01x02, U1 LM4040DBZ-2.0

Commit message: Final update
Routing:
- net GND: vias 324 -> 292
