File: Amplifier PCB.kicad_sch (KiCad schematic)
At the start: 20 parts, among them J1 sma, J2 sma, J3 Screw_Terminal_01x02, U1 LM4040DBZ-2.0

Commit message: Final update
Parts:
- DUT1: DIGIKEY 3157-PMA3-43-1W+CT-ND -> (none); MINI-CIRCUITS (none) -> PMA3-43-1W+
- L1, L2: Mouser (none) -> 994-0805LS-152XJRC; PARTNO (none) -> 0805LS-152XJRC
Changed lines of the file:
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@@
+			)
+		)
+		(property "PARTNO" "0805LS-152XJRC"
+			(at 179.07 90.17 0)
+			(effects
+				(font
+					(size 1.27 1.27)
+				)
+				(hide yes)
+			)
+		)
+		(property "Mouser" "994-0805LS-152XJRC"
+			(at 179.07 90.17 0)
+			(effects
+				(font
+					(size 1.27 1.27)
+				)
+				(hide yes)
 			)
 		)
@@
 			)
 		)
-		(property "PARTNO" ""
+		(property "PARTNO" "0805LS-152XJRC"
 			(at 121.92 111.76 0)
 			(effects
@@
 			)
 		)
-		(property "DIGIKEY" ""
+		(property "Mouser" "994-0805LS-152XJRC"
 			(at 121.92 111.76 0)
 			(effects
@@
 			)
 		)
-		(property "DIGIKEY" "3157-PMA3-43-1W+CT-ND"
+		(property "MINI-CIRCUITS" "PMA3-43-1W+"
 			(at 152.4 101.6 0)
 			(effects
